Commit message: Add body to xamyab robot

File: ur_description/urdf/xamyab_joint_limited_robot.urdf.xacro (robot description, xacro)
@@ -1,37 +1,5 @@
 <?xml version="1.0"?>
-<robot xmlns:xacro="http://wiki.ros.org/xacro"
-       name="xamyab" >
-  <!-- common stuff -->
-  <xacro:include filename="$(find ur_description)/urdf/common.gazebo.xacro" />
-  <!-- ur5 -->
-  <xacro:include filename="$(find ur_description)/urdf/xamyab.urdf.xacro" />
-  <!-- left arm -->
-  <xacro:ur5_robot prefix="left_" joint_limited="true"
-    shoulder_pan_lower_limit="${-pi}" shoulder_pan_upper_limit="${pi}"
-    shoulder_lift_lower_limit="${-pi}" shoulder_lift_upper_limit="${pi}"
-    elbow_joint_lower_limit="${-pi}" elbow_joint_upper_limit="${pi}"
-    wrist_1_lower_limit="${-pi}" wrist_1_upper_limit="${pi}"
-    wrist_2_lower_limit="${-pi}" wrist_2_upper_limit="${pi}"
-    wrist_3_lower_limit="${-pi}" wrist_3_upper_limit="${pi}"
-  />
-  <!-- right arm -->
-  <xacro:ur5_robot prefix="right_" joint_limited="true"
-    shoulder_pan_lower_limit="${-pi}" shoulder_pan_upper_limit="${pi}"
-    shoulder_lift_lower_limit="${-pi}" shoulder_lift_upper_limit="${pi}"
-    elbow_joint_lower_limit="${-pi}" elbow_joint_upper_limit="${pi}"
-    wrist_1_lower_limit="${-pi}" wrist_1_upper_limit="${pi}"
-    wrist_2_lower_limit="${-pi}" wrist_2_upper_limit="${pi}"
-    wrist_3_lower_limit="${-pi}" wrist_3_upper_limit="${pi}"
-  />
-  <link name="world" />
-  <joint name="left_world_joint" type="fixed">
-    <parent link="world" />
-    <child link = "left_base_link" />
-    <origin xyz="0.0 0.5 0.5" rpy="${-pi / 2} ${pi} 0.0" />
-  </joint>
-  <joint name="right_world_joint" type="fixed">
-    <parent link="world" />
-    <child link = "right_base_link" />
-    <origin xyz="0.0 -0.5 0.5" rpy="${pi / 2} 0.0 0.0" />
-  </joint>
+<robot xmlns:xacro="http://wiki.ros.org/xacro" name="xamyab_joint_limited_robot">
+    <xacro:include filename="$(find ur_description)/urdf/xamyab_robot.urdf.xacro"/>
+    <xacro:xamyab_robot joint_limited="true"/>
 </robot>

File: ur_description/urdf/xamyab_robot.urdf.xacro (robot description, xacro)
@@ -1,23 +1,58 @@
 <?xml version="1.0"?>
-<robot xmlns:xacro="http://wiki.ros.org/xacro"
-       name="xamyab" >
-  <!-- common stuff -->
-  <xacro:include filename="$(find ur_description)/urdf/common.gazebo.xacro" />
-  <!-- ur5 -->
-  <xacro:include filename="$(find ur_description)/urdf/xamyab.urdf.xacro" />
-  <!-- left arm -->
-  <xacro:ur5_robot prefix="left_" joint_limited="false"/>
-  <!-- right arm -->
-  <xacro:ur5_robot prefix="right_" joint_limited="false"/>
-  <link name="world" />
-  <joint name="world_joint" type="fixed">
-    <parent link="world" />
-    <child link = "left_base_link" />
-    <origin xyz="0.0 0.5 0.5" rpy="0.0 0.0 0.0" />
-  </joint>
-  <joint name="world_joint" type="fixed">
-    <parent link="world" />
-    <child link = "right_base_link" />
-    <origin xyz="0.0 -0.5 0.5" rpy="0.0 0.0 0.0" />
-  </joint>
+<robot xmlns:xacro="http://wiki.ros.org/xacro" name="xamyab">
+    <xacro:macro name="xamyab_robot" params="joint_limited:=false">
+        <!-- common stuff -->
+        <xacro:include filename="$(find ur_description)/urdf/common.gazebo.xacro"/>
+        <!-- ur5 -->
+        <xacro:include filename="$(find ur_description)/urdf/xamyab_ur5_arm.urdf.xacro"/>
+        <!-- body -->
+        <xacro:include filename="$(find ur_description)/urdf/xamyab_body.urdf.xacro"/>
+        <!-- left arm -->
+        <xacro:unless value="${joint_limited}">
+            <xacro:ur5_robot prefix="left_" joint_limited="false"/>
+        </xacro:unless>
+        <xacro:if value="${joint_limited}">
+            <xacro:ur5_robot prefix="left_" joint_limited="true"
+                             shoulder_pan_lower_limit="${-pi}" shoulder_pan_upper_limit="${pi}"
+                             shoulder_lift_lower_limit="${-pi}" shoulder_lift_upper_limit="${pi}"
+                             elbow_joint_lower_limit="${-pi}" elbow_joint_upper_limit="${pi}"
+                             wrist_1_lower_limit="${-pi}" wrist_1_upper_limit="${pi}"
+                             wrist_2_lower_limit="${-pi}" wrist_2_upper_limit="${pi}"
+                             wrist_3_lower_limit="${-pi}" wrist_3_upper_limit="${pi}"/>
+        </xacro:if>
+        <!-- right arm -->
+        <xacro:unless value="${joint_limited}">
+            <xacro:ur5_robot prefix="right_" joint_limited="false"/>
+        </xacro:unless>
+        <xacro:if value="${joint_limited}">
+            <xacro:ur5_robot prefix="right_" joint_limited="true"
+                             shoulder_pan_lower_limit="${-pi}" shoulder_pan_upper_limit="${pi}"
+                             shoulder_lift_lower_limit="${-pi}" shoulder_lift_upper_limit="${pi}"
+                             elbow_joint_lower_limit="${-pi}" elbow_joint_upper_limit="${pi}"
+                             wrist_1_lower_limit="${-pi}" wrist_1_upper_limit="${pi}"
+                             wrist_2_lower_limit="${-pi}" wrist_2_upper_limit="${pi}"
+                             wrist_3_lower_limit="${-pi}" wrist_3_upper_limit="${pi}"/>
+        </xacro:if>
+        <!-- arm body: Origin is the center of the bottom of the box -->
+        <xacro:property name="width" value="0.4"/>
+        <xacro:property name="depth" value="0.4"/>
+        <xacro:property name="height" value="0.6"/>
+        <xacro:xamyab_body width="${width}" depth="${depth}" height="${height}"/>
+        <link name="world"/>
+        <joint name="body_world_joint" type="fixed">
+            <parent link="world"/>
+            <child link="body_base_link"/>
+            <origin xyz="0.0 0.0 0.0" rpy="0.0 0.0 0.0"/>
+        </joint>
+        <joint name="left_world_joint" type="fixed">
+            <parent link="body_base_link"/>
+            <child link="left_base_link"/>
+            <origin xyz="${width / 2 * 0.6} ${depth / 2} ${height * 0.8}" rpy="${-pi / 2} ${pi} 0.0"/>
+        </joint>
+        <joint name="right_world_joint" type="fixed">
+            <parent link="body_base_link"/>
+            <child link="right_base_link"/>
+            <origin xyz="${width / 2 * 0.6} ${-depth / 2} ${height * 0.8}" rpy="${pi / 2} 0.0 0.0"/>
+        </joint>
+    </xacro:macro>
 </robot>
