Commit message: Update xamyab urdf model

File: ur_description/urdf/ground.urdf.xacro (robot description, xacro)
@@ -1,4 +1,4 @@
 <robot xmlns:xacro="http://wiki.ros.org/xacro" name="ground">
-    <xacro:macro name='ground' params="width:=${10.0} height:=${0.01} depth:=${10} mass:=${0.01}">
+    <xacro:macro name='ground' params="width:=${10.0} height:=${0.0001} depth:=${10} mass:=${0.01}">
         <xacro:property name="ixx" value="${1/12*mass*(height*height + depth*depth)}"/>
         <xacro:property name="iyy" value="${1/12*mass*(width*width + depth*depth)}"/>

File: ur_description/urdf/xamyab_robot.urdf.xacro (robot description, xacro)
@@ -2,6 +2,6 @@
 <robot xmlns:xacro="http://wiki.ros.org/xacro" name="xamyab">
     <xacro:arg name="limited" default="true"/>
-    <xacro:arg name="grippers" default="3"/>
-    <xacro:arg name="sim" default="true"/>
+    <xacro:arg name="grippers" default="0"/>
+    <xacro:arg name="sim" default="false"/>
     <xacro:property name="limited" value="$(arg limited)"/>
     <xacro:property name="grippers" value="$(arg grippers)"/>
@@ -55,5 +55,5 @@
         <xacro:property name="width" value="0.3048"/>
         <xacro:property name="depth" value="0.3048"/>
-        <xacro:property name="height" value="0.6096"/>
+        <xacro:property name="height" value="0.5755"/>
         <xacro:xamyab_body width="${width}" depth="${depth}" height="${height}"/>
         <link name="world"/>
@@ -61,5 +61,5 @@
             <parent link="world"/>
             <child link="ground_base_link"/>
-            <origin xyz="0 0 0.01" rpy="0 0 0"/>
+            <origin xyz="0 0 0.0001" rpy="0 0 0"/>
         </joint>
         <joint name="body_ground_joint" type="fixed">
