Commit message: Correct initial positions

File: ur_description/urdf/xamyab_robot.urdf.xacro (robot description, xacro)
@@ -5,5 +5,5 @@
         <xacro:include filename="$(find ur_description)/urdf/common.gazebo.xacro"/>
         <!-- ur5 -->
-        <xacro:include filename="$(find ur_description)/urdf/xamyab_ur5_arm.urdf.xacro"/>
+        <xacro:include filename="$(find ur_description)/urdf/ur5.urdf.xacro"/>
         <!-- body -->
         <xacro:include filename="$(find ur_description)/urdf/xamyab_body.urdf.xacro"/>
@@ -48,10 +48,10 @@
             <parent link="body_base_link"/>
             <child link="left_base_link"/>
-            <origin xyz="${width / 2 * 0.6} ${depth / 2} ${height * 0.8}" rpy="${-pi / 2} ${pi} 0.0"/>
+            <origin xyz="${width / 2 * 0.6} ${-depth / 2} ${height * .8}" rpy="${pi / 2} ${pi / 2} 0.0"/>
         </joint>
         <joint name="right_world_joint" type="fixed">
             <parent link="body_base_link"/>
             <child link="right_base_link"/>
-            <origin xyz="${width / 2 * 0.6} ${-depth / 2} ${height * 0.8}" rpy="${pi / 2} 0.0 0.0"/>
+            <origin xyz="${width / 2 * 0.6} ${depth / 2} ${height * .8}" rpy="${-pi / 2} ${-pi / 2} 0.0"/>
         </joint>
     </xacro:macro>

Commit message: Switch left to right arm

File: ur_description/urdf/xamyab_robot.urdf.xacro (robot description, xacro)
@@ -48,10 +48,10 @@
             <parent link="body_base_link"/>
             <child link="left_base_link"/>
-            <origin xyz="${width / 2 * 0.6} ${-depth / 2} ${height * .8}" rpy="${pi / 2} ${pi / 2} 0.0"/>
+            <origin xyz="${width / 2 * 0.6} ${depth / 2} ${height * .8}" rpy="${-pi / 2} ${-pi / 2} 0.0"/>
         </joint>
         <joint name="right_world_joint" type="fixed">
             <parent link="body_base_link"/>
             <child link="right_base_link"/>
-            <origin xyz="${width / 2 * 0.6} ${depth / 2} ${height * .8}" rpy="${-pi / 2} ${-pi / 2} 0.0"/>
+            <origin xyz="${width / 2 * 0.6} ${-depth / 2} ${height * .8}" rpy="${pi / 2} ${pi / 2} 0.0"/>
         </joint>
     </xacro:macro>

Commit message: Update xamyab size params

File: ur_description/urdf/xamyab_robot.urdf.xacro (robot description, xacro)
@@ -35,7 +35,7 @@
         </xacro:if>
         <!-- arm body: Origin is the center of the bottom of the box -->
-        <xacro:property name="width" value="0.4"/>
-        <xacro:property name="depth" value="0.4"/>
-        <xacro:property name="height" value="0.6"/>
+        <xacro:property name="width" value="0.3048"/>
+        <xacro:property name="depth" value="0.3048"/>
+        <xacro:property name="height" value="0.6096"/>
         <xacro:xamyab_body width="${width}" depth="${depth}" height="${height}"/>
         <link name="world"/>
@@ -48,10 +48,10 @@
             <parent link="body_base_link"/>
             <child link="left_base_link"/>
-            <origin xyz="${width / 2 * 0.6} ${depth / 2} ${height * .8}" rpy="${-pi / 2} ${-pi / 2} 0.0"/>
+            <origin xyz="${width / 2 - 0.105} ${depth / 2} 0.5334" rpy="${-pi / 2} ${-pi / 2} 0.0"/>
         </joint>
         <joint name="right_world_joint" type="fixed">
             <parent link="body_base_link"/>
             <child link="right_base_link"/>
-            <origin xyz="${width / 2 * 0.6} ${-depth / 2} ${height * .8}" rpy="${pi / 2} ${pi / 2} 0.0"/>
+            <origin xyz="${width / 2 - 0.105} ${-depth / 2} 0.5334" rpy="${pi / 2} ${pi / 2} 0.0"/>
         </joint>
     </xacro:macro>

Commit message: Add grippers to Gazebo and Refactor code

File: ur_description/urdf/xamyab_robot.urdf.xacro (robot description, xacro)
@@ -1,11 +1,22 @@
 <?xml version="1.0"?>
 <robot xmlns:xacro="http://wiki.ros.org/xacro" name="xamyab">
-    <xacro:macro name="xamyab_robot" params="joint_limited:=false">
-        <!-- common stuff -->
-        <xacro:include filename="$(find ur_description)/urdf/common.gazebo.xacro"/>
-        <!-- ur5 -->
-        <xacro:include filename="$(find ur_description)/urdf/ur5.urdf.xacro"/>
-        <!-- body -->
-        <xacro:include filename="$(find ur_description)/urdf/xamyab_body.urdf.xacro"/>
+    <xacro:arg name="limited" default="true"/>
+    <xacro:arg name="grippers" default="0"/>
+    <xacro:property name="limited" value="$(arg limited)"/>
+    <xacro:property name="grippers" value="$(arg grippers)"/>
+    <!--############## IMPORT STUFF ##############-->
+    <!-- common stuff -->
+    <xacro:include filename="$(find ur_description)/urdf/common.gazebo.xacro"/>
+    <!-- ur5 -->
+    <xacro:include filename="$(find ur_description)/urdf/ur5.urdf.xacro"/>
+    <!-- body -->
+    <xacro:include filename="$(find ur_description)/urdf/xamyab_body.urdf.xacro"/>
+    <!-- robotiq 2f 140 gripper -->
+    <xacro:if value="${grippers != 0}">
+        <xacro:include
+                filename="$(find robotiq_2f_140_gripper_visualization)/urdf/robotiq_arg2f_140_model_macro.xacro"/>
+    </xacro:if>
+    <xacro:macro name="xamyab_robot" params="joint_limited grippers">
+        <!--############## INITIALIZATION ##############-->
         <!-- left arm -->
         <xacro:unless value="${joint_limited}">
@@ -34,4 +45,5 @@
                              wrist_3_lower_limit="${-pi}" wrist_3_upper_limit="${pi}"/>
         </xacro:if>
+        <!--############## CONNECT LINKS ##############-->
         <!-- arm body: Origin is the center of the bottom of the box -->
         <xacro:property name="width" value="0.3048"/>
@@ -43,16 +55,35 @@
             <parent link="world"/>
             <child link="body_base_link"/>
-            <origin xyz="0.0 0.0 0.0" rpy="0.0 0.0 0.0"/>
+            <origin xyz="0 0 0" rpy="0 0 0"/>
         </joint>
-        <joint name="left_world_joint" type="fixed">
+        <joint name="left_body_joint" type="fixed">
             <parent link="body_base_link"/>
             <child link="left_base_link"/>
-            <origin xyz="${width / 2 - 0.105} ${depth / 2} 0.5334" rpy="${-pi / 2} ${-pi / 2} 0.0"/>
+            <origin xyz="${width / 2 - 0.105} ${depth / 2} 0.5334" rpy="${-pi / 2} ${-pi / 2} 0"/>
         </joint>
-        <joint name="right_world_joint" type="fixed">
+        <joint name="right_body_joint" type="fixed">
             <parent link="body_base_link"/>
             <child link="right_base_link"/>
-            <origin xyz="${width / 2 - 0.105} ${-depth / 2} 0.5334" rpy="${pi / 2} ${pi / 2} 0.0"/>
+            <origin xyz="${width / 2 - 0.105} ${-depth / 2} 0.5334" rpy="${pi / 2} ${pi / 2} 0"/>
         </joint>
+        <!-- left gripper -->
+        <xacro:if value="${grippers == 1 or grippers == 3}">
+            <xacro:robotiq_arg2f_140 prefix="lgripper_"/>
+            <joint name="lgripper_right_joint" type="fixed">
+                <parent link="left_tool0"/>
+                <child link="lgripper_robotiq_arg2f_base_link"/>
+                <origin xyz="0 0 0" rpy="0 0 0"/>
+            </joint>
+        </xacro:if>
+        <!-- right gripper -->
+        <xacro:if value="${grippers == 2 or grippers == 3}">
+            <xacro:robotiq_arg2f_140 prefix="rgripper_"/>
+            <joint name="rgripper_right_joint" type="fixed">
+                <parent link="right_tool0"/>
+                <child link="rgripper_robotiq_arg2f_base_link"/>
+                <origin xyz="0 0 0" rpy="0 0 0"/>
+            </joint>
+        </xacro:if>
     </xacro:macro>
+    <xacro:xamyab_robot joint_limited="${limited}" grippers="${grippers}"/>
 </robot>

Commit message: Add grippers for xamyab in Gazebo and MoveIt

File: ur_description/urdf/xamyab_robot.urdf.xacro (robot description, xacro)
@@ -2,5 +2,5 @@
 <robot xmlns:xacro="http://wiki.ros.org/xacro" name="xamyab">
     <xacro:arg name="limited" default="true"/>
-    <xacro:arg name="grippers" default="0"/>
+    <xacro:arg name="grippers" default="3"/>
     <xacro:property name="limited" value="$(arg limited)"/>
     <xacro:property name="grippers" value="$(arg grippers)"/>
@@ -70,5 +70,5 @@
         <xacro:if value="${grippers == 1 or grippers == 3}">
             <xacro:robotiq_arg2f_140 prefix="lgripper_"/>
-            <joint name="lgripper_right_joint" type="fixed">
+            <joint name="lgripper_left_joint" type="fixed">
                 <parent link="left_tool0"/>
                 <child link="lgripper_robotiq_arg2f_base_link"/>

Commit message: Add depth camera to gazebo

File: ur_description/urdf/xamyab_robot.urdf.xacro (robot description, xacro)
@@ -3,6 +3,8 @@
     <xacro:arg name="limited" default="true"/>
     <xacro:arg name="grippers" default="3"/>
+    <xacro:arg name="sim" default="true"/>
     <xacro:property name="limited" value="$(arg limited)"/>
     <xacro:property name="grippers" value="$(arg grippers)"/>
+    <xacro:property name="sim" value="true"/>
     <!--############## IMPORT STUFF ##############-->
     <!-- common stuff -->
@@ -85,4 +87,10 @@
             </joint>
         </xacro:if>
+        <!--Kinect-->
+        <xacro:if value="${sim}">
+            <!-- position of kinect has to be changed in common_sensors/urdf/sensors/kinect_properties.urdf.xacro-->
+            <xacro:include filename="$(find common_sensors)/urdf/sensors/kinect.urdf.xacro"/>
+            <xacro:sensor_kinect parent="body_base_link"/>
+        </xacro:if>
     </xacro:macro>
     <xacro:xamyab_robot joint_limited="${limited}" grippers="${grippers}"/>

Commit message: Add ground constraint to gazebo and fix spawning camera issue

File: ur_description/urdf/xamyab_robot.urdf.xacro (robot description, xacro)
@@ -6,8 +6,10 @@
     <xacro:property name="limited" value="$(arg limited)"/>
     <xacro:property name="grippers" value="$(arg grippers)"/>
-    <xacro:property name="sim" value="true"/>
+    <xacro:property name="sim" value="$(arg sim)"/>
     <!--############## IMPORT STUFF ##############-->
     <!-- common stuff -->
     <xacro:include filename="$(find ur_description)/urdf/common.gazebo.xacro"/>
+    <!-- ground -->
+    <xacro:include filename="$(find ur_description)/urdf/ground.urdf.xacro"/>
     <!-- ur5 -->
     <xacro:include filename="$(find ur_description)/urdf/ur5.urdf.xacro"/>
@@ -21,4 +23,6 @@
     <xacro:macro name="xamyab_robot" params="joint_limited grippers">
         <!--############## INITIALIZATION ##############-->
+        <!--ground -->
+        <xacro:ground/>
         <!-- left arm -->
         <xacro:unless value="${joint_limited}">
@@ -54,6 +58,11 @@
         <xacro:xamyab_body width="${width}" depth="${depth}" height="${height}"/>
         <link name="world"/>
-        <joint name="body_world_joint" type="fixed">
+        <joint name="ground_world_joint" type="fixed">
             <parent link="world"/>
+            <child link="ground_base_link"/>
+            <origin xyz="0 0 0.01" rpy="0 0 0"/>
+        </joint>
+        <joint name="body_ground_joint" type="fixed">
+            <parent link="ground_base_link"/>
             <child link="body_base_link"/>
             <origin xyz="0 0 0" rpy="0 0 0"/>

Commit message: Update xamyab urdf model

File: ur_description/urdf/xamyab_robot.urdf.xacro (robot description, xacro)
@@ -71,10 +71,10 @@
             <parent link="body_base_link"/>
             <child link="left_base_link"/>
-            <origin xyz="${width / 2 - 0.105} ${depth / 2} 0.5334" rpy="${-pi / 2} ${-pi / 2} 0"/>
+            <origin xyz="${width / 2 - 0.105} ${depth / 2} 0.5134" rpy="${-pi / 2} ${-pi / 2} 0"/>
         </joint>
         <joint name="right_body_joint" type="fixed">
             <parent link="body_base_link"/>
             <child link="right_base_link"/>
-            <origin xyz="${width / 2 - 0.105} ${-depth / 2} 0.5334" rpy="${pi / 2} ${pi / 2} 0"/>
+            <origin xyz="${width / 2 - 0.105} ${-depth / 2} 0.5134" rpy="${pi / 2} ${pi / 2} 0"/>
         </joint>
         <!-- left gripper -->

Commit message: Update Xamyab model to match the real robot

File: ur_description/urdf/xamyab_robot.urdf.xacro (robot description, xacro)
@@ -93,5 +93,5 @@
                 <parent link="right_tool0"/>
                 <child link="rgripper_robotiq_arg2f_base_link"/>
-                <origin xyz="0 0 0" rpy="0 0 0"/>
+                <origin xyz="0 0 0" rpy="0 0 ${pi / 2}"/>
             </joint>
         </xacro:if>
